File: board/bitsyled-v1.sch (EAGLE design)
At the start: 8 parts

Commit message: Updatez
Connections:
- removed net VCC: D1.A
- net 5V: now also D1.A
- net VR: now also D1.C
Other:
- moved on the sheet: D1
Changed lines of the file:
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@@
 <instance part="OTHER" gate="G$1" x="-17.78" y="81.28"/>
 <instance part="C1" gate="G$1" x="10.16" y="68.58"/>
-<instance part="D1" gate="G$1" x="5.08" y="76.2"/>
+<instance part="D1" gate="G$1" x="2.54" y="83.82"/>
 </instances>
 <busses>
@@
 <junction x="-39.37" y="27.94"/>
 <label x="-39.37" y="17.78" size="1.778" layer="95" xref="yes"/>
+</segment>
+<segment>
+<pinref part="D1" gate="G$1" pin="A"/>
+<wire x1="0" y1="83.82" x2="0" y2="76.2" width="0.1524" layer="91"/>
+<label x="0" y="76.2" size="1.778" layer="95" rot="R180" xref="yes"/>
 </segment>
 </net>
@@
 </segment>
 </net>
-<net name="N$3" class="0">
-<segment>
-<wire x1="27.94" y1="25.4" x2="43.18" y2="25.4" width="0.1524" layer="91"/>
-</segment>
-</net>
-<net name="N$6" class="0">
-<segment>
-<wire x1="27.94" y1="17.78" x2="43.18" y2="17.78" width="0.1524" layer="91"/>
-</segment>
-</net>
 <net name="VR" class="0">
 <segment>
@@
 <junction x="10.16" y="76.2"/>
 <label x="17.78" y="76.2" size="1.778" layer="95" rot="MR180" xref="yes"/>
+<pinref part="D1" gate="G$1" pin="C"/>
+<wire x1="5.08" y1="83.82" x2="7.62" y2="83.82" width="0.1524" layer="91"/>
+<wire x1="7.62" y1="83.82" x2="7.62" y2="76.2" width="0.1524" layer="91"/>
 </segment>
 </net>
-<net name="VCC" class="0">
-<segment>
-<pinref part="D1" gate="G$1" pin="A"/>
-<wire x1="2.54" y1="76.2" x2="0" y2="76.2" width="0.1524" layer="91"/>
-<label x="0" y="76.2" size="1.778" layer="95" rot="R180" xref="yes"/>
-</segment>
-</net>
