File: board/bitsyled-v1.2.1.brd (EAGLE design)
At the start: 16 x 14.2 mm, 8 parts

Commit message: updates
Parts:
- moved R1 3.82 mm to (14.7, 8.01), turned to 90 degrees
- moved LED1 2.85 mm to (11.3, 7.87), turned to 90 degrees
- moved C1 1.59 mm to (14.7, 10.0), turned to 270 degrees
- moved CPU 1.01 mm to (7.52, 10.2), turned to 180 degrees
- moved D1 0.63 mm to (1.55, 9.86)
Routing:
- net 5V: track 0.00 -> 57.5 mm, vias 0 -> 1
- net GND: track 0.00 -> 48.8 mm, vias 0 -> 2
- net LD1: track 0.00 -> 19.3 mm, vias 0 -> 1
- net SDA: track 0.00 -> 17.8 mm
- net VR: track 0.00 -> 16.2 mm
- net RESET: track 0.00 -> 13.3 mm
- net LD0: track 0.00 -> 11.0 mm, vias 0 -> 1
- net BLED: track 0.00 -> 9.90 mm, vias 0 -> 1
- net LD2: track 0.00 -> 8.86 mm, vias 0 -> 1
- net MISO: track 0.00 -> 8.71 mm
- net RC: track 0.00 -> 6.33 mm, vias 0 -> 1
- net SCL: track 0.00 -> 5.52 mm
- net N$2: track 0.00 -> 2.85 mm
