File: board/bitsyled-v1.2.1.brd (EAGLE design)
At the start: 16 x 14.2 mm, 8 parts

Commit message: Adding presets
Parts:
- C1: value (none) -> 10uf
- R1: value (none) -> 140
Changed lines of the file:
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@@
 <?xml version="1.0" encoding="utf-8"?>
 <!DOCTYPE eagle SYSTEM "eagle.dtd">
-<eagle version="8.3.2">
+<eagle version="9.3.2">
 <drawing>
 <settings>
-<setting alwaysvectorfont="no"/>
+<setting alwaysvectorfont="yes"/>
 <setting verticaltext="up"/>
 </settings>
@@
 <layer number="59" name="tCarbon" color="7" fill="1" visible="no" active="no"/>
 <layer number="60" name="bCarbon" color="7" fill="1" visible="no" active="no"/>
-<layer number="88" name="SimResults" color="9" fill="1" visible="no" active="yes"/>
-<layer number="89" name="SimProbes" color="9" fill="1" visible="no" active="yes"/>
+<layer number="88" name="SimResults" color="9" fill="1" visible="no" active="no"/>
+<layer number="89" name="SimProbes" color="9" fill="1" visible="no" active="no"/>
 <layer number="90" name="Modules" color="5" fill="1" visible="no" active="no"/>
 <layer number="91" name="Nets" color="2" fill="1" visible="no" active="no"/>
@@
 <param name="dpMaxLengthDifference" value="10mm"/>
 <param name="dpGapFactor" value="2.5"/>
-<param name="checkGrid" value="0"/>
 <param name="checkAngle" value="0"/>
 <param name="checkFont" value="1"/>
 <param name="checkRestrict" value="1"/>
+<param name="checkStop" value="0"/>
+<param name="checkValues" value="0"/>
+<param name="checkNames" value="1"/>
+<param name="checkWireStubs" value="1"/>
+<param name="checkPolygonWidth" value="0"/>
 <param name="useDiameter" value="13"/>
 <param name="maxErrors" value="50"/>
@@
 <attribute name="VALUE" value="ATTINY84" x="7.5216" y="10.2476" size="1.778" layer="28" rot="MR180" display="off"/>
 </element>
-<element name="C1" library="adafruit" package="C0805" value="" x="14.6812" y="10.0208" smashed="yes" rot="MR270">
+<element name="C1" library="adafruit" package="C0805" value="10uf" x="14.6812" y="10.0208" smashed="yes" rot="MR270">
 <attribute name="VALUE" x="16.9672" y="10.9098" size="1.27" layer="28" rot="MR270"/>
 </element>
@@
 <attribute name="VALUE" x="13.0718" y="9.271" size="0.4064" layer="27" ratio="10" rot="R180"/>
 </element>
-<element name="R1" library="microbuilder" package="_0805" value="" x="14.73" y="8.0122" smashed="yes" rot="R90">
+<element name="R1" library="microbuilder" package="_0805" value="140" x="14.73" y="8.0122" smashed="yes" rot="R90">
 <attribute name="VALUE" x="16.381" y="6.4248" size="0.4064" layer="27" ratio="10" rot="R90"/>
 </element>
-<element name="RL0" library="FPVTools" package="BITSYLED_1X6_RAIL" value="BITSYLED_1X6_RAILNORMAL" x="15.63" y="3.635"/>
-<element name="RL1" library="FPVTools" package="BITSYLED_1X6_RAIL_R" value="BITSYLED_1X6_RAILREVERSED" x="15.63" y="13.16"/>
-<element name="PRG" library="FPVTools" package="BITSYLED_1X6_RAIL_PRG" value="BITSYLED_1X6_RAILPRG" x="15.63" y="3.635"/>
+<element name="RL0" library="FPVTools" package="BITSYLED_1X6_RAIL" value="BITSYLED_1X6_RAILNORMAL" x="15.63" y="3.635" smashed="yes"/>
+<element name="RL1" library="FPVTools" package="BITSYLED_1X6_RAIL_R" value="BITSYLED_1X6_RAILREVERSED" x="15.63" y="13.16" smashed="yes"/>
+<element name="PRG" library="FPVTools" package="BITSYLED_1X6_RAIL_PRG" value="BITSYLED_1X6_RAILPRG" x="15.63" y="3.635" smashed="yes"/>
 </elements>
 <signals>
@@
 </signal>
 </signals>
+<mfgpreviewcolors>
+<mfgpreviewcolor name="soldermaskcolor" color="0xC8008000"/>
+<mfgpreviewcolor name="silkscreencolor" color="0xFFFEFEFE"/>
+<mfgpreviewcolor name="backgroundcolor" color="0xFF282828"/>
+<mfgpreviewcolor name="coppercolor" color="0xFFFFBF00"/>
+<mfgpreviewcolor name="substratecolor" color="0xFF786E46"/>
+</mfgpreviewcolors>
 <errors>
 </errors>
